Commit message: Updated urdf
Fix the arrow keys problem

File: src/drive/urdf/drive3.urdf (robot description, URDF)
Before this commit: robot drive, 16 links, 15 joints
Joints:
- joint imu_joint: origin xyz=0.30 -0.30 1.13 rpy=0 0 0 -> xyz=0.30 0 0.30 rpy=0 0 0
- joint joint_wheel_4: axis 0.99619 -0.014024 -0.08602 -> -0.99619 0.014024 0.08602
- joint joint_wheel_5: axis 0.99619 -0.014024 -0.08602 -> -0.99619 0.014024 0.08602
- joint joint_wheel_6: axis 0.99619 -0.014024 -0.08602 -> -0.99619 0.014024 0.08602
- joint lidar_joint: origin xyz=0.25 0 1.13 rpy=0 0 0 -> xyz=0.25 0 0.60 rpy=0 0 0

Commit message: Update joint origins for imu and lidar links
Imu and lidar joints updated

File: src/drive/urdf/drive3.urdf (robot description, URDF)
Before this commit: robot drive, 16 links, 15 joints
Joints:
- joint imu_joint: origin xyz=0.30 0 0.30 rpy=0 0 0 -> xyz=0.30 -0.40 1.13 rpy=0 0 0
- joint lidar_joint: origin xyz=0.25 0 0.60 rpy=0 0 0 -> xyz=0.25 -0.38 1.13 rpy=0 0 0

Commit message: Slam done

File: src/drive/urdf/drive3.urdf (robot description, URDF)
Before this commit: robot drive, 16 links, 15 joints
Joints:
- joint base_joint: origin xyz=0 0 1 rpy=0 3.1416 0 -> xyz=0 0 0.398 rpy=0 3.1416 0
- joint imu_joint: origin xyz=0.30 -0.40 1.13 rpy=0 0 0 -> xyz=0.30 -0.40 0.52 rpy=0 0 0
- joint lidar_joint: origin xyz=0.25 -0.38 1.13 rpy=0 0 0 -> xyz=0.25 -0.38 0.52 rpy=0 0 0

Commit message: Nav2 Implemented

File: src/drive/urdf/drive3.urdf (robot description, URDF)
Before this commit: robot drive, 16 links, 15 joints
Links:
- link imu_link: geometry 
- link lidar_link: mass 0.01 -> 0.1; geometry collision cylinder length=0.04 radius=0.03; visual cylinder length=0.04 radius=0.03
Joints:
- joint base_joint: origin xyz=0 0 0.398 rpy=0 3.1416 0 -> xyz=0 0 0.398 rpy=0 3.1416 1.5708
- joint imu_joint: origin xyz=0.30 -0.40 0.52 rpy=0 0 0 -> xyz=0 0 0 rpy=0 0 0
- joint joint_wheel_1: limit lower=-1000000 upper=1000000 effort=1000 velocity=1000 -> (none); type revolute -> continuous
- joint joint_wheel_2: limit lower=-1000000 upper=1000000 effort=1000 velocity=1000 -> (none); type revolute -> continuous
- joint joint_wheel_3: limit lower=-1000000 upper=1000000 effort=1000 velocity=1000 -> (none); type revolute -> continuous
- joint joint_wheel_4: limit lower=-1000000 upper=1000000 effort=1000 velocity=1000 -> (none); type revolute -> continuous
- joint joint_wheel_5: limit lower=-1000000 upper=1000000 effort=1000 velocity=1000 -> (none); type revolute -> continuous
- joint joint_wheel_6: limit lower=-1000000 upper=1000000 effort=1000 velocity=1000 -> (none); type revolute -> continuous
- joint lidar_joint: origin xyz=0.25 -0.38 0.52 rpy=0 0 0 -> xyz=0.32 0.33 0.55 rpy=0 0 0

Commit message: Rtabmap Nav2

File: src/drive/urdf/drive3.urdf (robot description, URDF)
Before this commit: robot drive, 16 links, 15 joints
Links:
- removed link lidar_link
- added link camera_link, mass 0.1; collision box size=0.04 0.08 0.04; visual box size=0.04 0.08 0.04
- added link camera_optical_link
Joints:
- removed joint lidar_joint
- added joint camera_joint: type fixed, parent base_link, child camera_link, origin xyz=0.32 0.33 0.55 rpy=0 0 0
- added joint camera_optical_joint: type fixed, parent camera_link, child camera_optical_link, origin xyz=0 0 0 rpy=-1.5708 0 -1.5708

Commit message: Nav2 with rtabmap implemente

File: src/drive/urdf/drive3.urdf (robot description, URDF)
Before this commit: robot drive, 17 links, 16 joints
Joints:
- joint camera_joint: origin xyz=0.32 0.33 0.55 rpy=0 0 0 -> xyz=0.52 0.30 0.55 rpy=0 0.2618 0
